File: PCB/NotSmart-Speaker/NotSmart-Speaker.kicad_pcb (KiCad board)
At the start: 4 copper layers, 100 x 100 mm, 102 parts, among them IC1 FUSB302TMPX, IC2 TPA3118D2DAPR, J1 UJ20-C-H-G-SMT-2-P16-TR, J2 Screw_Terminal_01x02, SW1 TS04-66-43-BK-160-SMT, SW2 TS04-66-43-BK-160-SMT, U1 ESP32-S3-WROOM-1, U2 USBLC6-2SC6, U3 AP2112K-3.3, U4 SN74LV1T34DBV, U5 AP2112K-3.3, U6 TPS62933, U7 PCM5100A

Commit message: V1.1
Parts:
- C34, C35, C36, C37: footprint Capacitor_SMD:C_0805_2012Metric_Pad1.18x1.45mm_HandSolder -> Capacitor_SMD:C_1206_3216Metric_Pad1.33x1.80mm_HandSolder
