File: PCB/NotSmart-Speaker/NotSmart-Speaker.kicad_sch (KiCad schematic)
At the start: 58 parts, among them IC1 FUSB302TMPX, J1 UJ20-C-H-G-SMT-2-P16-TR, J2 Screw_Terminal_01x02, SW1 TS04-66-43-BK-160-SMT, SW2 TS04-66-43-BK-160-SMT, U1 ESP32-S3-WROOM-1, U2 USBLC6-2SC6, U3 AP2112K-3.3, U4 SN74LV1T34DBV, U5 AP2112K-3.3, U6 TPS62933

Commit message: V1.1
Parts:
- C1, C2, C4, C5, C6, C9: Manufacturer_Part_Number (none) -> GRM219R61H105MA73D
- C10: Manufacturer_Part_Number (none) -> 885012207095
- C11, C3, C7: Manufacturer_Part_Number (none) -> 885012207098R
- C12: Manufacturer_Part_Number (none) -> 08055A180JAT4A
- C13: Manufacturer_Part_Number (none) -> MLASL21GBB5476MTNA01
- C8: Manufacturer_Part_Number (none) -> GRM21BR61H106KE43K
- D4, D5: Manufacturer_Part_Number (none) -> LTST-S220KGKT
- D6: Manufacturer_Part_Number (none) -> LTST-C171YKT
- D8: Manufacturer_Part_Number (none) -> 150080BS75000
- J1: Manufacturer_Part_Number (none) -> UJ20-C-H-G-SMT-2-P16-TR
- J2: Manufacturer_Part_Number (none) -> 1751248
- R1, R4, R5: Manufacturer_Part_Number (none) -> RC0805FR-0710KL
- R10, R11, R14, R15: Manufacturer_Part_Number (none) -> AC0805FR-101KL
- R12: Manufacturer_Part_Number (none) -> ERJ-PB6B4302V
- R13: Manufacturer_Part_Number (none) -> ERJ-PB6B8201V
- R2, R3: Manufacturer_Part_Number (none) -> CRCW08050000ZSTC
- R6, R7, R8: Manufacturer_Part_Number (none) -> CR0805-FX-4701ELF
- R9: Manufacturer_Part_Number (none) -> CRCW0805330RJNEA
- TP1, TP2, TP3, TP4, TP5: now not fitted; now left out of the parts list
- U1: Manufacturer_Part_Number (none) -> ESP32-S3-WROOM-1-N8R8
- U2: Manufacturer_Part_Number (none) -> USBLC6-2SC6
- U3, U5: Manufacturer_Part_Number (none) -> 621-AP2112K-3.3TRG1
- U4: Manufacturer_Part_Number (none) -> SN74LV1T34DBVRG4
- U6: Manufacturer_Part_Number (none) -> TPS62933ODRLR
