File: PCB/NotSmart-Speaker/audio.kicad_sch (KiCad schematic)
At the start: 43 parts, among them IC2 TPA3118D2DAPR, U7 PCM5100A

Commit message: V1.1
Parts:
- C14, C16, C20, C21, C24, C25, C32, C33: value 0.1u -> 100n; Manufacturer_Part_Number (none) -> 885012207098R
- C15, C17, C22, C23: Manufacturer_Part_Number (none) -> GRM21BR61H106KE43K
- C18, C19: Manufacturer_Part_Number (none) -> CL21B225KAFNNNE
- C26, C27: Manufacturer_Part_Number (none) -> GRM219R61H105MA73D
- C28, C29, C30, C31: Manufacturer_Part_Number (none) -> CL21B225KBYNNWE
- C34, C35: Manufacturer_Part_Number (none) -> GRM31CR71E106MA12L
- C36, C37: Manufacturer_Part_Number (none) -> 885012208092
- C38, C39: Manufacturer_Part_Number (none) -> EEH-ZS1H221P
- C40, C41: Manufacturer_Part_Number (none) -> 885012207086
- C42, C43: Manufacturer_Part_Number (none) -> 08055C103KAT2A
- R16, R17, R20, R22: Manufacturer_Part_Number (none) -> RC0805FR-0710KL
- R18, R19: Manufacturer_Part_Number (none) -> CR0805-JW-471ELF
- R21: Manufacturer_Part_Number (none) -> CRCW080512K0JNEA
- R24: Manufacturer_Part_Number (none) -> CRCW08050000ZSTC
- U7: Manufacturer_Part_Number (none) -> PCM5100APWR
